File: Report Schematic/Port Expander for Plug and Play.sch (EAGLE design)
At the start: 6 parts, among them IC1 MCP23017SO, IC3 MCP23017SO

Commit message: Schematics for manual
Parts:
- removed IC3: MCP23017SO, adafruit:MCP23017SO
- removed JP2, JP6: (no value), adafruit:PINHD-1X8BIG
Connections:
- removed net INTAB: IC3.INTA, IC3.INTB
- removed net N$10: IC3.GPA4, JP5.5
- removed net N$2: IC3.GPA0, JP5.1
- removed net N$23: IC3.GPA5, JP5.6
- removed net N$32: IC3.GPA6, JP5.7
- removed net N$33: IC3.GPA7, JP5.8
- removed net N$34: IC3.GPB0, JP6.1
- removed net N$35: IC3.GPB1, JP6.2
- removed net N$36: IC3.GPB2, JP6.3
- removed net N$37: IC3.GPB3, JP6.4
- removed net N$38: IC3.GPB4, JP6.5
- removed net N$39: IC3.GPB5, JP6.6
- removed net N$40: IC3.GPB6, JP6.7
- removed net N$41: IC3.GPB7, JP6.8
- removed net N$5: IC3.GPA1, JP5.2
- removed net N$8: IC3.GPA2, JP5.3
- removed net N$9: IC3.GPA3, JP5.4
- removed net RST: IC3.!RESET
- removed net SCL: IC3.SCL
- removed net SDA: IC3.SDA
- net 3.3V: no longer IC3.A0, IC3.A1, IC3.A2, IC3.VDD, IC3.VSS
- net N$14: now also JP5.1; no longer JP2.1
- net N$15: now also JP5.2; no longer JP2.2
- net N$16: now also JP5.3; no longer JP2.3
- net N$17: now also JP5.4; no longer JP2.4
- net N$18: now also JP5.5; no longer JP2.5
- net N$19: now also JP5.6; no longer JP2.6
- net N$20: now also JP5.7; no longer JP2.7
- net N$21: now also JP5.8; no longer JP2.8
Other:
- note removed: "Interrupt To uC on Pin 29 PF1"
- note removed: "SCL going to I2C0SCL of uC on Pin 47 PB2"
- note removed: "SDA going to I2C0SDA of uC on Pin 48 PB3"
- moved on the sheet: IC1, JP4, JP5
