File: Report Schematic/Reset Switch.sch (EAGLE design)
At the start: 12 parts, among them U2 LMV358, U3 LMV324

Commit message: Schematics for manual
Parts:
- removed R10, R13, R15, R17, R19: 33K, adafruit:R-US_M1206
- removed R11, R12, R14, R16, R18: 22K, adafruit:R-US_M1206
- removed U2: LMV358, SparkFun-IC-Amplifiers:LMV358SOIC
- removed U3: LMV324, SparkFun-IC-Amplifiers:LMV324
- added C9: 2.2uF, SparkFun-Capacitors:2.2UF-1206-50V-10%
- added R1: 10K, adafruit:R-US_M1206
- added S1: Push Button, SparkFun-Switches:MOMENTARY-SWITCH-SPST-PTH-6.0MM
Connections:
- removed net 11: U2G1.+IN
- removed net 15: U3G1.+IN
- removed net 41: U3G2.+IN
- removed net 44: U3G3.+IN
- removed net 45: U3G4.+IN
- removed net EX1: R12.1, R13.1
- removed net EX6: R16.1, R17.1
- removed net GND: R10.2, R13.2, R15.2, R17.2, R19.2
- removed net N1: R11.2, U2G1.-IN, U2G1.OUT
- removed net N2: R12.2, U3G1.-IN, U3G1.OUT
- removed net N3: R14.2, U3G2.-IN, U3G2.OUT
- removed net N4: R16.2, U3G3.-IN, U3G3.OUT
- removed net N5: R18.2, U3G4.-IN, U3G4.OUT
- removed net PB4: R10.1, R11.1
- removed net PD2: R14.1, R15.1
- removed net PE4: R18.1, R19.1
- new net 3.3V: C9.2
- new net RST: C9.1, R1.2, S1.1
- new net VDD: R1.1
Other:
- note added: "3.3V Supply"
- note added: "Connected to reset of uC on pin 38"
- note removed: "Connected to 1st channel of External ADC"
- note removed: "Connected to 6th channel of External ADC"
- note removed: "Connected to PB4"
- note removed: "Connected to PD2"
- note removed: "Connected to PE4"
- note removed: "Plug and Play Board"
- note removed: "Sharp IR2 ,Pin 15 on Main Board"
- note removed: "Sharp IR3 ,Pin 41 on Main Board"
- note removed: "Sharp IR4 ,Pin 20 on Main Board"
- note removed: "Sharp IR4 ,Pin 44 on Main Board"
- note removed: "Sharp IR5 ,Pin 45 on Main Board"
