File: Schematic 2/Schematic-1.brd (EAGLE design)
At the start: 126.3 x 83.1 mm, 37 parts, among them IC1 7805T, IC3 MCP23017SO, Q1 BSS138, Q2 BSS138, U2 LMV358, U3 LMV324

Commit message: Adding groung to layout of plugable TIVA board
Routing:
- net 5V2: track 70.9 -> 71.4 mm, vias 5 -> 4
- added copper zone on layer 1, net GND
- added copper zone on layer 16, net GND
Changed lines of the file:
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@@
 <wire x1="4.2" y1="36.9" x2="4.179" y2="36.931" width="0.2" layer="1"/>
 <wire x1="6.7" y1="36.9" x2="6.719" y2="36.931" width="0.2" layer="1"/>
-<wire x1="10.6316" y1="34.2709" x2="11.3687" y2="34.2709" width="0.2" layer="1"/>
-<wire x1="11.3687" y1="34.2709" x2="11.3897" y2="34.2499" width="0.2" layer="1"/>
-<via x="11.3897" y="34.2499" extent="1-16" drill="0.35"/>
-<wire x1="11.3897" y1="34.2499" x2="13.0687" y2="34.2499" width="0.2" layer="16"/>
+<via x="10.1226" y="34.2499" extent="1-16" drill="0.35"/>
 <wire x1="13.0687" y1="34.2499" x2="14.1642" y2="35.3454" width="0.2" layer="16"/>
 <wire x1="14.1642" y1="35.3454" x2="14.7848" y2="35.3454" width="0.2" layer="16"/>
@@
 <wire x1="24.2655" y1="37.3933" x2="26.2933" y2="37.3933" width="0.2" layer="1"/>
 <wire x1="26.2933" y1="37.3933" x2="26.3" y2="37.4" width="0.2" layer="1"/>
-<wire x1="9.7161" y1="36.931" x2="10.1742" y2="36.4729" width="0.2" layer="1"/>
-<wire x1="10.1742" y1="36.4729" x2="10.1742" y2="34.7283" width="0.2" layer="1"/>
-<wire x1="10.1742" y1="34.7283" x2="10.6316" y2="34.2709" width="0.2" layer="1"/>
-<wire x1="6.719" y1="36.931" x2="9.7161" y2="36.931" width="0.2" layer="1"/>
+<wire x1="6.719" y1="36.931" x2="8.5762" y2="36.931" width="0.2" layer="1"/>
+<wire x1="8.5762" y1="36.931" x2="9.0409" y2="36.4663" width="0.2" layer="1"/>
+<wire x1="9.0409" y1="36.4663" x2="9.0409" y2="34.5251" width="0.2" layer="1"/>
+<wire x1="9.0409" y1="34.5251" x2="9.3063" y2="34.2597" width="0.2" layer="1"/>
+<wire x1="9.3063" y1="34.2597" x2="10.1128" y2="34.2597" width="0.2" layer="1"/>
+<wire x1="10.1128" y1="34.2597" x2="10.1226" y2="34.2499" width="0.2" layer="1"/>
+<wire x1="10.1226" y1="34.2499" x2="13.0687" y2="34.2499" width="0.2" layer="16"/>
 </signal>
 <signal name="13">
@@
 <wire x1="99.6963" y1="3.2399" x2="100.7" y2="4.2436" width="1.016" layer="16"/>
 <wire x1="100.7" y1="4.2436" x2="100.7" y2="5" width="1.016" layer="16"/>
+<polygon width="0.1524" layer="1">
+<vertex x="-10" y="70"/>
+<vertex x="-10" y="-30"/>
+<vertex x="130" y="-30"/>
+<vertex x="130" y="70"/>
+<vertex x="-10" y="70"/>
+</polygon>
+<polygon width="0.1524" layer="16">
+<vertex x="-20" y="75"/>
+<vertex x="-20" y="-35"/>
+<vertex x="135" y="-35"/>
+<vertex x="135" y="75"/>
+</polygon>
 </signal>
 <signal name="PF1">
@@
 <contactref element="U$1" pad="10"/>
 <contactref element="U$2" pad="VBUS"/>
-<wire x1="47.75" y1="30.177" x2="50.5162" y2="30.177" width="0.2" layer="1"/>
-<wire x1="50.5162" y1="30.177" x2="51.6122" y2="31.273" width="0.2" layer="1"/>
-<wire x1="51.6122" y1="31.273" x2="51.6122" y2="32.6931" width="0.2" layer="1"/>
 <wire x1="51.6122" y1="32.6931" x2="51.6752" y2="32.7561" width="0.2" layer="1"/>
 <via x="51.6752" y="32.7561" extent="1-16" drill="0.35"/>
-<wire x1="51.6752" y1="32.7561" x2="51.6752" y2="34.2711" width="0.2" layer="16"/>
-<wire x1="51.6752" y1="34.2711" x2="50.855" y2="35.0913" width="0.2" layer="16"/>
+<wire x1="50.855" y1="35.0913" x2="51.18465" y2="34.76165" width="0.2" layer="16"/>
 <via x="50.855" y="35.0913" extent="1-16" drill="0.35"/>
-<wire x1="50.855" y1="35.0913" x2="46.0009" y2="35.0913" width="0.2" layer="1"/>
-<wire x1="46.0009" y1="35.0913" x2="36.7646" y2="44.3276" width="0.2" layer="1"/>
-<wire x1="36.7646" y1="44.3276" x2="11.1918" y2="44.3276" width="0.2" layer="1"/>
+<wire x1="45.681" y1="35.4112" x2="45.55295" y2="35.53925" width="0.2" layer="1"/>
 <wire x1="11.1918" y1="44.3276" x2="10.9514" y2="44.0872" width="0.2" layer="1"/>
 <via x="10.9514" y="44.0872" extent="1-16" drill="0.35"/>
-<wire x1="10.9514" y1="38.0876" x2="10.9514" y2="44.0872" width="0.2" layer="16"/>
-<wire x1="8.4977" y1="31.851" x2="6.719" y2="31.851" width="0.2" layer="16"/>
-<wire x1="10.9194" y1="37.9968" x2="10.8969" y2="37.9743" width="0.2" layer="16"/>
 <via x="10.8969" y="37.9743" extent="1-16" drill="0.35"/>
-<wire x1="10.8969" y1="37.9743" x2="10.8969" y2="35.6009" width="0.2" layer="1"/>
-<wire x1="10.8969" y1="35.6009" x2="11.262" y2="35.2358" width="0.2" layer="1"/>
-<wire x1="11.262" y1="35.2358" x2="12.1745" y2="35.2358" width="0.2" layer="1"/>
-<wire x1="12.1745" y1="35.2358" x2="12.5579" y2="34.8524" width="0.2" layer="1"/>
-<wire x1="12.5579" y1="34.8524" x2="12.5579" y2="33.0083" width="0.2" layer="1"/>
-<wire x1="12.5579" y1="33.0083" x2="11.8461" y2="32.2965" width="0.2" layer="1"/>
-<via x="11.8461" y="32.2965" extent="1-16" drill="0.35"/>
-<wire x1="11.8461" y1="32.2965" x2="8.9432" y2="32.2965" width="0.2" layer="16"/>
-<wire x1="8.9432" y1="32.2965" x2="8.4977" y2="31.851" width="0.2" layer="16"/>
-<wire x1="10.9194" y1="37.9968" x2="10.9514" y2="38.0876" width="0" layer="19" extent="16-16"/>
+<wire x1="10.9514" y1="43.4024" x2="10.9514" y2="43.6792" width="0.2" layer="16"/>
+<wire x1="47.75" y1="30.177" x2="50.3896" y2="30.177" width="1.016" layer="1"/>
+<wire x1="50.3896" y1="30.177" x2="51.6122" y2="31.3996" width="1.016" layer="1"/>
+<wire x1="51.6122" y1="31.3996" x2="51.6122" y2="32.6931" width="1.016" layer="1"/>
+<wire x1="50.855" y1="35.0913" x2="50.5351" y2="35.4112" width="1.016" layer="1"/>
+<wire x1="50.5351" y1="35.4112" x2="45.681" y2="35.4112" width="1.016" layer="1"/>
+<wire x1="45.55295" y1="35.53925" x2="36.7646" y2="44.3276" width="1.016" layer="1"/>
+<wire x1="36.7646" y1="44.3276" x2="11.1918" y2="44.3276" width="1.016" layer="1"/>
+<wire x1="10.9514" y1="43.4024" x2="10.8969" y2="43.3479" width="1.016" layer="16"/>
+<wire x1="10.8969" y1="43.3479" x2="10.8969" y2="37.9743" width="1.016" layer="16"/>
+<wire x1="10.9514" y1="43.6792" x2="10.9514" y2="44.0872" width="1.016" layer="16"/>
+<wire x1="10.9888" y1="37.8824" x2="10.8969" y2="37.9743" width="1.016" layer="1"/>
+<wire x1="50.855" y1="33.5763" x2="50.855" y2="35.0913" width="1.016" layer="16"/>
+<wire x1="51.6752" y1="32.7561" x2="50.855" y2="33.5763" width="1.016" layer="16"/>
+<wire x1="10.8969" y1="37.9743" x2="10.2131" y2="37.2905" width="1.016" layer="1"/>
+<wire x1="10.2131" y1="37.2905" x2="10.2131" y2="36.1554" width="1.016" layer="1"/>
+<wire x1="12.0098" y1="34.3587" x2="10.2131" y2="36.1554" width="1.016" layer="1"/>
+<wire x1="6.719" y1="31.851" x2="6.9451" y2="31.6249" width="1.016" layer="1"/>
+<wire x1="11.4592" y1="31.6249" x2="12.0098" y2="32.1755" width="1.016" layer="1"/>
+<wire x1="12.0098" y1="32.1755" x2="12.0098" y2="34.3587" width="1.016" layer="1"/>
+<wire x1="6.9451" y1="31.6249" x2="11.4592" y2="31.6249" width="1.016" layer="1"/>
 </signal>
 <signal name="N$9">

Commit message: Plugable TIVA changes on 13-06-17
Parts:
- added U$3: SELF-LOCKING_SWITCHSELF-LOCKING_SWITCH, Switch_Self-locking:SELF-LOCKING_SWITCH
- moved IC1 21.7 mm to (15.9, -12.0)
- moved C1 19.8 mm to (24.9, 0.53)
- moved C2 17.3 mm to (16.0, 1.66)
- moved JP1 16.7 mm to (20.1, 10.0)
- moved JP3 16.7 mm to (20.1, 15.4)
- moved JP2 16.7 mm to (20.1, 12.7)
- moved JP6 8.57 mm to (32.5, -8.20)
- moved JP7 8.57 mm to (29.8, -8.20)
Connections:
- new net 5V2': U$2.VBUS, U$3.2B
- new net GND': U$2.GND, U$3.1B
- net 5V2: now also U$3.2A; no longer U$2.VBUS
- net GND: now also U$3.1A; no longer U$2.GND, U$2.GND'
Routing:
- net GND': track 0.00 -> 69.7 mm, vias 0 -> 2
- net 22: track 145.1 -> 78.4 mm
- net 5V2': track 0.00 -> 61.5 mm, vias 0 -> 2
- net 37: track 74.3 -> 129.3 mm, vias 2 -> 0
- net 5V2: track 71.4 -> 29.5 mm, vias 4 -> 1
- net SCL: track 146.1 -> 106.2 mm, vias 3 -> 5
- net 69: track 121.4 -> 161.2 mm, vias 4 -> 1
- net GND: track 326.3 -> 292.5 mm, vias 11 -> 12
- net 36: track 106.8 -> 73.8 mm, vias 0 -> 2
- net 32: track 74.6 -> 42.8 mm, vias 2 -> 1
- net 44: track 70.3 -> 39.3 mm, vias 0 -> 2
- net N$19: track 78.2 -> 98.6 mm, vias 2 -> 8
- net PB2: track 34.8 -> 54.4 mm
- net 12V: track 47.2 -> 66.8 mm, vias 4 -> 2
- net 5V-SERVO: track 37.2 -> 21.4 mm
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Other:
- board text added: "1A"
- board text added: "2A"

Commit message: Version 2 of Plug and Play Board
Parts:
- added LED1, LED10, LED11, LED12, LED13, LED14, LED15, LED16, LED2, LED3, LED4, LED5, LED6, LED7, LED8, LED9: (no value), adafruit:1206
- moved JP7 21.2 mm to (26.4, 12.7)
- moved JP6 19.2 mm to (26.4, 10.0), turned to 180 degrees
- moved U$2 15.5 mm to (74.7, 20.8), turned to 180 degrees
- moved U2 13.1 mm to (96.9, 6.72)
- moved IC1 9.87 mm to (6.39, -14.8), turned to 140 degrees
- moved R1 8.94 mm to (61.6, 3.22), turned to 180 degrees
- moved R3 8.54 mm to (61.7, 9.09)
- moved C1 4.76 mm to (22.0, -3.22)
- moved C2 3.72 mm to (17.1, -1.89)
- moved JP4 2.73 mm to (35.3, -8.87)
- moved JP5 2.42 mm to (99.3, -8.38)
- moved IC3 2.15 mm to (66.8, -12.2)
- moved R4 1.82 mm to (54.4, 3.00), turned to 90 degrees
- moved U$3 1.61 mm to (3.49, 5.49)
Connections:
- net 5V2: now also U$3.2C; no longer U$3.2A
- net GND: now also LED1.C, LED10.C, LED11.C, LED12.C, LED13.C, LED14.C, LED15.C, LED16.C, LED2.C, LED3.C, LED4.C, LED5.C, LED6.C, LED7.C, LED8.C, LED9.C
- net N$10: now also LED5.A
- net N$11: now also LED6.A
- net N$12: now also LED7.A
- net N$15: now also LED8.A
- net N$20: now also LED9.A
- net N$21: now also LED10.A
- net N$22: now also LED11.A
- net N$23: now also LED12.A
- net N$24: now also LED13.A
- net N$25: now also LED15.A
- net N$28: now also LED14.A
- net N$29: now also LED16.A
- net N$3: now also LED1.A
- net N$7: now also LED3.A
- net N$8: now also LED4.A
- net N$9: now also LED2.A
Routing:
- net 53: track 38.5 -> 146.4 mm, vias 0 -> 2
- net PB2: track 54.4 -> 153.6 mm, vias 1 -> 3
- net PF0: track 41.8 -> 138.5 mm
- net 50: track 30.9 -> 123.2 mm, vias 0 -> 4
- net 71: track 39.5 -> 124.7 mm, vias 0 -> 2
- net 12: track 42.4 -> 126.1 mm, vias 0 -> 1
- net 16: track 75.4 -> 148.8 mm
- net 45: track 126.9 -> 55.1 mm, vias 2 -> 1
- net 70: track 35.1 -> 102.7 mm, vias 0 -> 4
- net PF1: track 34.5 -> 101.0 mm, vias 0 -> 2
- net 26: track 82.9 -> 17.5 mm, vias 2 -> 0
- net 13: track 51.2 -> 115.5 mm, vias 0 -> 3
- net SCL: track 106.2 -> 169.4 mm, vias 5 -> 9
- net PB7: track 86.3 -> 23.6 mm, vias 5 -> 0
- net 37: track 129.3 -> 67.5 mm, vias 0 -> 2
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Other:
- outline, holes or cut-outs redrawn
- board text added: "Developed by ERTS Lab"
- board text added: "PF4"
- board text added: "PORTA"
- board text added: "PORTB"
- board text added: "Signal"
- board text added: "Version 2.0"
- board text removed: "PORT A"
- board text removed: "PORT B"
